File: Kicad/Switch/Switch.kicad_pcb (KiCad board)
At the start: 2 copper layers, 63.5 x 53.3 mm, 18 parts, among them Q1 BD139, Q2 IXTH90P10P, Q4 BD139, Q5A1 BSC340N08NS3G, Q6 BD139

Commit message: Vp1 socket
install Vp1 socket
Parts:
- added V8: Conn_01x01_Socket, Connector_PinSocket_1.27mm:PinSocket_1x01_P1.27mm_Vertical, F.Cu at (147.3, 81.3)
Connections:
- net +1V8 renamed Net-(V8-Pin_1)
Routing:
- net Net-(V8-Pin_1): track 15.2 -> 21.0 mm
Changed lines of the file:
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@@
   (net 8 "Net-(Q2-S)")
   (net 9 "Net-(Q4-E)")
-  (net 10 "+1V8")
+  (net 10 "Net-(V8-Pin_1)")
   (net 11 "Net-(Q4-B)")
   (footprint "Package_TO_SOT_THT:TO-92_Inline" (layer "F.Cu")
@@
       (stroke (width 0.1) (type solid)) (layer "F.Fab"))
     (pad "1" smd roundrect (at -1.4625 0 270) (size 1.125 2.65) (layers "F.Cu" "F.Paste" "F.Mask") (roundrect_rratio 0.222222)
-      (net 10 "+1V8") (pintype "passive"))
+      (net 10 "Net-(V8-Pin_1)") (pintype "passive"))
     (pad "2" smd roundrect (at 1.4625 0 270) (size 1.125 2.65) (layers "F.Cu" "F.Paste" "F.Mask") (roundrect_rratio 0.222222)
       (net 5 "Net-(D2-K)") (pintype "passive"))
@@
       (net 1 "Net-(C19-Pad1)") (pintype "passive"))
     (model "${KICAD6_3DMODEL_DIR}/Resistor_SMD.3dshapes/R_0805_2012Metric.wrl"
+      (offset (xyz 0 0 0))
+      (scale (xyz 1 1 1))
+      (rotate (xyz 0 0 0))
+    )
+  )
+  (footprint "Connector_PinSocket_1.27mm:PinSocket_1x01_P1.27mm_Vertical" (layer "F.Cu")
+    (at 147.32 81.28)
+    (descr "Through hole straight socket strip, 1x01, 1.27mm pitch, single row (from Kicad 4.0.7), script generated")
+    (tags "Through hole socket strip THT 1x01 1.27mm single row")
+    (property "Sheetfile" "Switch.kicad_sch")
+    (property "Sheetname" "")
+    (property "ki_description" "Generic connector, single row, 01x01, script generated")
+    (property "ki_keywords" "connector")
+    (attr through_hole)
+    (fp_text reference "V8" (at 0 -2.135) (layer "F.SilkS")
+        (effects (font (size 1 1) (thickness 0.15)))
+    )
+    (fp_text value "Conn_01x01_Socket" (at 0 2.135) (layer "F.Fab")
+        (effects (font (size 1 1) (thickness 0.15)))
+    )
+    (fp_text user "${REFERENCE}" (at 0 0) (layer "F.Fab")
+        (effects (font (size 0.76 0.76) (thickness 0.11)))
+    )
+    (fp_line (start -1.33 0.575) (end -1.33 0.695)
+      (stroke (width 0.12) (type solid)) (layer "F.SilkS"))
+    (fp_line (start -1.33 0.695) (end -0.76 0.695)
+      (stroke (width 0.12) (type solid)) (layer "F.SilkS"))
+    (fp_line (start 0 -0.76) (end 1.33 -0.76)
+      (stroke (width 0.12) (type solid)) (layer "F.SilkS"))
+    (fp_line (start 0.76 0.695) (end 1.33 0.695)
+      (stroke (width 0.12) (type solid)) (layer "F.SilkS"))
+    (fp_line (start 1.33 -0.76) (end 1.33 0)
+      (stroke (width 0.12) (type solid)) (layer "F.SilkS"))
+    (fp_line (start 1.33 0.575) (end 1.33 0.695)
+      (stroke (width 0.12) (type solid)) (layer "F.SilkS"))
+    (fp_line (start -1.8 -1.15) (end 1.75 -1.15)
+      (stroke (width 0.05) (type solid)) (layer "F.CrtYd"))
+    (fp_line (start -1.8 1.15) (end -1.8 -1.15)
+      (stroke (width 0.05) (type solid)) (layer "F.CrtYd"))
+    (fp_line (start 1.75 -1.15) (end 1.75 1.15)
+      (stroke (width 0.05) (type solid)) (layer "F.CrtYd"))
+    (fp_line (start 1.75 1.15) (end -1.8 1.15)
+      (stroke (width 0.05) (type solid)) (layer "F.CrtYd"))
+    (fp_line (start -1.27 -0.635) (end 0.9525 -0.635)
+      (stroke (width 0.1) (type solid)) (layer "F.Fab"))
+    (fp_line (start -1.27 0.635) (end -1.27 -0.635)
+      (stroke (width 0.1) (type solid)) (layer "F.Fab"))
+    (fp_line (start 0.9525 -0.635) (end 1.27 -0.3175)
+      (stroke (width 0.1) (type solid)) (layer "F.Fab"))
+    (fp_line (start 1.27 -0.3175) (end 1.27 0.635)
+      (stroke (width 0.1) (type solid)) (layer "F.Fab"))
+    (fp_line (start 1.27 0.635) (end -1.27 0.635)
+      (stroke (width 0.1) (type solid)) (layer "F.Fab"))
+    (pad "1" thru_hole rect (at 0 0) (size 1 1) (drill 0.7) (layers "*.Cu" "*.Mask")
+      (net 10 "Net-(V8-Pin_1)") (pinfunction "Pin_1") (pintype "passive"))
+    (model "${KICAD6_3DMODEL_DIR}/Connector_PinSocket_1.27mm.3dshapes/PinSocket_1x01_P1.27mm_Vertical.wrl"
       (offset (xyz 0 0 0))
       (scale (xyz 1 1 1))
@@
       (stroke (width 0.1) (type solid)) (layer "F.Fab"))
     (pad "1" smd roundrect (at -1.4625 0 270) (size 1.125 2.65) (layers "F.Cu" "F.Paste" "F.Mask") (roundrect_rratio 0.222222)
-      (net 10 "+1V8") (pintype "passive"))
+      (net 10 "Net-(V8-Pin_1)") (pintype "passive"))
     (pad "2" smd roundrect (at 1.4625 0 270) (size 1.125 2.65) (layers "F.Cu" "F.Paste" "F.Mask") (roundrect_rratio 0.222222)
       (net 5 "Net-(D2-K)") (pintype "passive"))
@@
       (stroke (width 0.1) (type solid)) (layer "F.Fab"))
     (pad "1" smd roundrect (at -1.4625 0 270) (size 1.125 2.65) (layers "F.Cu" "F.Paste" "F.Mask") (roundrect_rratio 0.222222)
-      (net 10 "+1V8") (pintype "passive"))
+      (net 10 "Net-(V8-Pin_1)") (pintype "passive"))
     (pad "2" smd roundrect (at 1.4625 0 270) (size 1.125 2.65) (layers "F.Cu" "F.Paste" "F.Mask") (roundrect_rratio 0.222222)
       (net 5 "Net-(D2-K)") (pintype "passive"))
@@
   (segment (start 129.54 78.74) (end 135.6975 78.74) (width 0.25) (layer "F.Cu") (net 9))
   (segment (start 134.62 85.975) (end 142.24 85.975) (width 0.25) (layer "F.Cu") (net 10))
-  (segment (start 149.86 85.975) (end 142.24 85.975) (width 0.25) (layer "F.Cu") (net 10))
+  (segment (start 147.32 83.435) (end 144.78 85.975) (width 0.25) (layer "F.Cu") (net 10))
+  (segment (start 149.86 85.975) (end 144.78 85.975) (width 0.25) (layer "F.Cu") (net 10))
+  (segment (start 144.78 85.975) (end 142.24 85.975) (width 0.25) (layer "F.Cu") (net 10))
+  (segment (start 147.32 81.28) (end 147.32 83.435) (width 0.25) (layer "F.Cu") (net 10))
   (segment (start 124.46 73.66) (end 124.46 76.2) (width 0.25) (layer "F.Cu") (net 11))
   (segment (start 121.92 96.52) (end 127.715 96.52) (width 0.25) (layer "F.Cu") (net 11))

Commit message: update
Routing:
- net Net-(D1-K): track 42.4 -> 49.0 mm
- net Net-(D1-A): track 33.5 -> 30.2 mm
- net Net-(Q1-C): track 53.1 -> 56.1 mm
Changed lines of the file:
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@@
   )
   (setup
+    (stackup
+      (layer "F.SilkS" (type "Top Silk Screen"))
+      (layer "F.Paste" (type "Top Solder Paste"))
+      (layer "F.Mask" (type "Top Solder Mask") (thickness 0.01))
+      (layer "F.Cu" (type "copper") (thickness 0.035))
+      (layer "dielectric 1" (type "core") (thickness 1.51) (material "FR4") (epsilon_r 4.5) (loss_tangent 0.02))
+      (layer "B.Cu" (type "copper") (thickness 0.035))
+      (layer "B.Mask" (type "Bottom Solder Mask") (thickness 0.01))
+      (layer "B.Paste" (type "Bottom Solder Paste"))
+      (layer "B.SilkS" (type "Bottom Silk Screen"))
+      (copper_finish "None")
+      (dielectric_constraints no)
+    )
     (pad_to_mask_clearance 0)
     (pcbplotparams
@@
   (segment (start 170.18 65.54) (end 170.18 71.76) (width 0.25) (layer "F.Cu") (net 1))
   (segment (start 170.745 65.54) (end 170.68 65.54) (width 0.25) (layer "F.Cu") (net 1))
-  (segment (start 142.24 60.96) (end 137.16 60.96) (width 0.25) (layer "F.Cu") (net 3))
   (segment (start 127 68.58) (end 127 66.04) (width 0.25) (layer "F.Cu") (net 3))
-  (segment (start 129.54 68.58) (end 127 68.58) (width 0.25) (layer "F.Cu") (net 3))
+  (segment (start 142.24 60.96) (end 139.7 63.5) (width 0.25) (layer "F.Cu") (net 3))
+  (segment (start 139.7 63.5) (end 139.7 71.12) (width 0.25) (layer "F.Cu") (net 3))
+  (segment (start 139.7 71.12) (end 129.54 71.12) (width 0.25) (layer "F.Cu") (net 3))
+  (segment (start 129.54 71.12) (end 127 68.58) (width 0.25) (layer "F.Cu") (net 3))
   (segment (start 138.3 73.66) (end 127 73.66) (width 0.25) (layer "F.Cu") (net 3))
   (segment (start 127 78.74) (end 127 68.58) (width 0.25) (layer "F.Cu") (net 3))
-  (segment (start 137.16 60.96) (end 129.54 68.58) (width 0.25) (layer "F.Cu") (net 3))
-  (segment (start 156.21 72.39) (end 154.94 73.66) (width 0.25) (layer "F.Cu") (net 4))
+  (segment (start 148.785 64.575) (end 142.24 71.12) (width 0.25) (layer "F.Cu") (net 4))
+  (segment (start 156.21 63.5) (end 155.79 63.92) (width 0.25) (layer "F.Cu") (net 4))
   (segment (start 142.24 73.66) (end 139.7 73.66) (width 0.25) (layer "F.Cu") (net 4))
   (segment (start 142.24 66.04) (end 142.24 73.66) (width 0.25) (layer "F.Cu") (net 4))
-  (segment (start 156.21 63.5) (end 156.21 72.39) (width 0.25) (layer "F.Cu") (net 4))
-  (segment (start 154.94 73.66) (end 142.24 73.66) (width 0.25) (layer "F.Cu") (net 4))
-  (segment (start 162.56 96.52) (end 162.56 88.9) (width 0.25) (layer "F.Cu") (net 5))
+  (segment (start 142.24 71.12) (end 142.24 73.66) (width 0.25) (layer "F.Cu") (net 4))
+  (segment (start 155.79 63.92) (end 155.79 64.575) (width 0.25) (layer "F.Cu") (net 4))
+  (segment (start 155.79 64.575) (end 148.785 64.575) (width 0.25) (layer "F.Cu") (net 4))
   (segment (start 142.24 88.9) (end 134.62 88.9) (width 0.25) (layer "F.Cu") (net 5))
   (segment (start 175.26 94.905) (end 173.28 92.925) (width 0.25) (layer "F.Cu") (net 5))
   (segment (start 162.56 96.735) (end 162.56 99.06) (width 0.25) (layer "F.Cu") (net 5))
-  (segment (start 154.94 88.9) (end 149.86 88.9) (width 0.25) (layer "F.Cu") (net 5))
-  (segment (start 149.86 93.98) (end 154.94 88.9) (width 0.25) (layer "F.Cu") (net 5))
+  (segment (start 152.4 93.98) (end 157.48 88.9) (width 0.25) (layer "F.Cu") (net 5))
+  (segment (start 149.86 93.98) (end 152.4 93.98) (width 0.25) (layer "F.Cu") (net 5))
   (segment (start 162.56 99.06) (end 175.26 99.06) (width 0.25) (layer "F.Cu") (net 5))
+  (segment (start 162.56 96.52) (end 162.56 93.98) (width 0.25) (layer "F.Cu") (net 5))
   (segment (start 162.56 96.735) (end 162.56 96.52) (width 0.25) (layer "F.Cu") (net 5))
   (segment (start 157.695 96.735) (end 157.48 96.52) (width 0.25) (layer "F.Cu") (net 5))
   (segment (start 157.48 96.52) (end 162.56 96.52) (width 0.25) (layer "F.Cu") (net 5))
-  (segment (start 162.56 88.9) (end 154.94 88.9) (width 0.25) (layer "F.Cu") (net 5))
   (segment (start 149.86 88.9) (end 142.24 88.9) (width 0.25) (layer "F.Cu") (net 5))
   (segment (start 175.26 99.06) (end 175.26 94.905) (width 0.25) (layer "F.Cu") (net 5))
+  (segment (start 162.56 93.98) (end 157.48 88.9) (width 0.25) (layer "F.Cu") (net 5))
+  (segment (start 157.48 88.9) (end 149.86 88.9) (width 0.25) (layer "F.Cu") (net 5))
   (segment (start 149.86 96.52) (end 129.54 96.52) (width 0.25) (layer "F.Cu") (net 6))
   (segment (start 157.48 93.98) (end 154.94 96.52) (width 0.25) (layer "F.Cu") (net 6))
   (segment (start 154.94 96.52) (end 149.86 96.52) (width 0.25) (layer "F.Cu") (net 6))
   (segment (start 149.86 95.38) (end 149.86 96.52) (width 0.25) (layer "F.Cu") (net 6))
+  (segment (start 142.24 63.5) (end 149.86 63.5) (width 0.25) (layer "F.Cu") (net 7))
   (segment (start 149.86 58.42) (end 154.94 63.5) (width 0.25) (layer "F.Cu") (net 7))
   (segment (start 127 55.88) (end 147.32 55.88) (width 0.25) (layer "F.Cu") (net 7))
-  (segment (start 142.24 63.5) (end 147.32 58.42) (width 0.25) (layer "F.Cu") (net 7))
   (segment (start 127 55.88) (end 124.46 55.88) (width 0.25) (layer "F.Cu") (net 7))
-  (segment (start 147.32 58.42) (end 149.86 58.42) (width 0.25) (layer "F.Cu") (net 7))
   (segment (start 127 63.115) (end 127 55.88) (width 0.25) (layer "F.Cu") (net 7))
   (segment (start 147.32 55.88) (end 149.86 58.42) (width 0.25) (layer "F.Cu") (net 7))
+  (segment (start 149.86 63.5) (end 149.86 58.42) (width 0.25) (layer "F.Cu") (net 7))
   (segment (start 124.46 55.88) (end 124.46 58.42) (width 0.25) (layer "F.Cu") (net 7))
   (segment (start 165.1 93.53) (end 166.4 94.83) (width 0.25) (layer "F.Cu") (net 8))
