File: KiCad/Switch7.0/Switch.kicad_sch (KiCad schematic)
At the start: 20 parts, among them J1 Conn_01x01, Q1 BD139, Q2 IXTH90P10P, Q4 BD139, Q5A1 BSC340N08NS3G, Q6 BD139

Commit message: new version update
Parts:
- removed V56, V8, VTackt1, Vout1: Conn_01x01_Socket, Connector_PinSocket_1.27mm:PinSocket_1x01_P1.27mm_Vertical, symbol Connector:Conn_01x01_Socket
- added J2, J3, J4, J5: Conn_01x01, Connector:Banana_Jack_1Pin, symbol Connector_Generic:Conn_01x01
- Q2: footprint Package_TO_SOT_THT:TO-92_Inline -> Library:TO-247-PMOS
Connections:
- net GND: now also J5.1 (Pin_1)
- net at Q2.3 (S), Q5A1.5 (D), R23.1: now also J4.1 (Pin_1)
- net Power: now reaches Q1.2 (C), Q2.1 (D), R2.1
- net Power: now also J1.1 (Pin_1)
- net at R22.1, R58.1, R59.1: now also J2.1 (Pin_1)
- net at Q4.3 (B), R25.2: now also J3.1 (Pin_1)
Other:
- moved on the sheet: J1
