File: KiCad/Switch6.0/Switch6.0.kicad_pcb (KiCad board)
At the start: 2 copper layers, 128 x 90 mm, 20 parts, among them Q1 BD139, Q2 IXTH90P10P, Q4 BD139, Q5A1 BSC340N08NS3G, Q6 BD139

Commit message: Final results
Parts:
- added C10: 0.1uF, Capacitor_SMD:C_0805_2012Metric, F.Cu at (189.0, 49.2)
- added C11: 0.1uF, Capacitor_SMD:C_0805_2012Metric, F.Cu at (196.0, 49.2)
- added C2: 0.1uF, Capacitor_SMD:C_0805_2012Metric, F.Cu at (133.0, 49.2)
- added C3: 0.1uF, Capacitor_SMD:C_0805_2012Metric, F.Cu at (140.0, 49.2)
- added C4: 0.1uF, Capacitor_SMD:C_0805_2012Metric, F.Cu at (147.0, 49.2)
- added C5: 0.1uF, Capacitor_SMD:C_0805_2012Metric, F.Cu at (154.0, 49.2)
- added C6: 0.1uF, Capacitor_SMD:C_0805_2012Metric, F.Cu at (161.0, 49.5)
- added C7: 0.1uF, Capacitor_SMD:C_0805_2012Metric, F.Cu at (168.0, 49.2)
- added C8: 0.1uF, Capacitor_SMD:C_0805_2012Metric, F.Cu at (175.0, 49.3)
- added C9: 0.1uF, Capacitor_SMD:C_0805_2012Metric, F.Cu at (182.0, 49.2)
- added Q_D1: Conn_01x01, Connector_PinHeader_2.54mm:PinHeader_1x01_P2.54mm_Vertical, F.Cu at (196.0, 99.0)
- added Q_G1: Conn_01x01, Connector_PinHeader_2.54mm:PinHeader_1x01_P2.54mm_Vertical, F.Cu at (155.0, 91.0)
- added Q_G2: Conn_01x01, Connector_PinHeader_2.54mm:PinHeader_1x01_P2.54mm_Vertical, F.Cu at (186.0, 120.0)
- added Q_Masse1: Conn_01x01, Connector_PinHeader_2.54mm:PinHeader_1x01_P2.54mm_Vertical, F.Cu at (196.0, 70.0)
- added Q_S1: Conn_01x01, Connector_PinHeader_2.54mm:PinHeader_1x01_P2.54mm_Vertical, F.Cu at (163.0, 83.0)
- added R10: 2R2, Resistor_SMD:R_2512_6332Metric, F.Cu at (182.0, 58.0)
- added R11: 2R2, Resistor_SMD:R_2512_6332Metric, F.Cu at (189.0, 58.0)
- added R12: 2R2, Resistor_SMD:R_2512_6332Metric, F.Cu at (196.0, 58.0)
- added R3: 2R2, Resistor_SMD:R_2512_6332Metric, F.Cu at (133.0, 58.0)
- added R4: 2R2, Resistor_SMD:R_2512_6332Metric, F.Cu at (140.0, 58.0)
- added R5: 2R2, Resistor_SMD:R_2512_6332Metric, F.Cu at (147.0, 58.0)
- added R6: 2R2, Resistor_SMD:R_2512_6332Metric, F.Cu at (154.0, 58.0)
- added R7: 2R2, Resistor_SMD:R_2512_6332Metric, F.Cu at (161.0, 58.0)
- added R8: 2R2, Resistor_SMD:R_2512_6332Metric, F.Cu at (168.0, 58.0)
- added R9: 2R2, Resistor_SMD:R_2512_6332Metric, F.Cu at (175.0, 58.0)
- moved VTackt1 25.2 mm to (124.0, 91.0)
- moved R25 1.00 mm to (126.0, 125.1)
Connections:
- net Net-(D1-Pad1) renamed G1
- net Net-(D8-Pad2) renamed G2
Routing:
- net 56V: track 78.3 -> 237.3 mm
- net GND: track 50.6 -> 119.9 mm, vias 4 -> 7
- net D: track 63.0 -> 78.3 mm
- net G2: track 74.4 -> 82.6 mm
- net Tackt: track 41.6 -> 34.5 mm
- net G1: track 40.9 -> 47.1 mm
- net Net-(C5-Pad1): track 0.00 -> 4.29 mm
- net Net-(C4-Pad1): track 0.00 -> 4.29 mm
- net Net-(C3-Pad1): track 0.00 -> 4.29 mm
- net Net-(C2-Pad1): track 0.00 -> 4.29 mm
- net Net-(C9-Pad1): track 0.00 -> 4.04 mm
- net Net-(C8-Pad1): track 0.00 -> 4.04 mm
- net Net-(C7-Pad1): track 0.00 -> 4.04 mm
- net Net-(C6-Pad1): track 0.00 -> 4.04 mm
- net Net-(C11-Pad1): track 0.00 -> 4.04 mm
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Other:
- board size 128 x 90 mm -> 107 x 109.2 mm
- board text added: "Switch Ver 0.1 FH Dortmund Mohamad Sayad"
- board text removed: "Switch ver 0.1 FH Dortmund Mohamad Sayad"

Commit message: Simulation and Kicad update
Simulation oof the Switch updated with an op amp. Kicad structure updated (0.2 version)
Parts:
- renumbered V56 to +56V_in, Vout1 to +56V_out, Vp8 to +5V_in, GNDall1 to GND, VTackt1 to Gate
Routing:
- net GND: track 119.9 -> 113.6 mm, vias 7 -> 13
- net 56V: track 237.3 -> 241.4 mm
- added copper zone on F.Cu, net 56V
Other:
- board text added: "Switch Ver 0.2 FH Dortmund Mohamad Sayad"
- board text removed: "Switch Ver 0.1 FH Dortmund Mohamad Sayad"

Commit message: Switch Platine
Platine 0.2 Entwurf mit OpV
Parts:
- removed Gate: Conn_01x01, Connector:Banana_Jack_1Pin
- added R1.1: 10k, Resistor_SMD:R_0805_2012Metric, F.Cu at (119.7, 73.5)
- added R1.2: 2k, Resistor_SMD:R_0805_2012Metric, F.Cu at (113.2, 73.5)
- added U1: AD8033, Package_SO:SOIC-8_3.9x4.9mm_P1.27mm, F.Cu at (114.7, 63.4)
- added V_Gate: Conn_01x01, Connector:Banana_Jack_1Pin, F.Cu at (98.7, 77.2)
- D1, D8: value BAT54XV2T5G -> type="D" model="BAT54XV2T5G" lib=""
- moved Q_G1 6.61 mm to (148.4, 91.3)
- moved Q_S1 5.53 mm to (164.2, 77.6)
- moved Q_Masse1 1.49 mm to (197.4, 70.5)
- moved +56V_in 0.71 mm to (181.9, 71.7)
- moved +56V_out 0.61 mm to (208.4, 108.9)
- moved GND 0.36 mm to (172.8, 140.7)
- moved +5V_in 0.30 mm to (140.7, 106.5)
Connections:
- net Tackt renamed Net-(Q4-B)
Routing:
- net GND: track 113.6 -> 144.9 mm
- net Net-(Q4-B): track 34.5 -> 63.5 mm
- net Net-(U1--): track 0.00 -> 27.7 mm, vias 0 -> 2
- net Tackt: track 0.00 -> 20.7 mm
- net G2: track 82.9 -> 86.5 mm
- net 56V: track 241.4 -> 243.4 mm
- net G1: track 47.1 -> 46.4 mm
- added copper zone on F.Cu, net Net-(Q4-B)
- added copper zone on F.Cu, net Net-(U1--)
- added copper zone on F.Cu, net Tackt
Other:
- board size 107 x 109.2 mm -> 128.8 x 109.2 mm
