File: KiCad/Switch/Switch.kicad_pcb (KiCad board)
At the start: 2 copper layers, 128.8 x 109.2 mm, 48 parts, among them Q1 BD139, Q2 IXTH90P10P, Q4 BD139, Q5A1 BSC340N08NS3G, Q6 BD139, U1 AD8033

Commit message: Simulation und PCB update
Parts:
- added +24V_in: Conn_01x01, Connector:Banana_Jack_1Pin, F.Cu at (98.8, 49.8)
- moved Q_D1 5.20 mm to (196.1, 93.8)
- renumbered V_Gate to V_gate
Connections:
- U1 pad 7: 56V -> Net-(U1-V+)
Routing:
- net Net-(U1-V+): track 0.00 -> 31.2 mm
- net GND: track 144.9 -> 116.5 mm, vias 13 -> 12
- net 56V: track 243.4 -> 235.8 mm
- net D: track 78.3 -> 83.6 mm
- added copper zone on F.Cu, net Net-(U1-V+)

Commit message: kicad switch LDO install
Parts:
- removed +24V_in: Conn_01x01, Connector:Banana_Jack_1Pin
- added Clod1: 0.1uF, Capacitor_SMD:C_0805_2012Metric, F.Cu at (125.3, 56.0)
- added Clod2: 0.1uF, Capacitor_SMD:C_0805_2012Metric, F.Cu at (124.0, 61.2)
- added Rlod1: 1.35k, Resistor_SMD:R_0805_2012Metric, F.Cu at (120.2, 52.6)
- added Rlod2: 25.2k, Resistor_SMD:R_0805_2012Metric, F.Cu at (120.2, 57.9)
- added U2: LT3014, Package_TO_SOT_SMD:SOT-23-5, F.Cu at (125.8, 47.3)
- renumbered GND to GNDall1, +56V_in to V56, V_gate to VTackt1, +56V_out to Vout1, +5V_in to Vp8
Routing:
- net Net-(U2-ADJ): track 0.00 -> 23.7 mm
- net 56V: track 235.8 -> 257.7 mm
- net GND: track 116.5 -> 133.4 mm, vias 12 -> 14
- net Net-(U1-V+): track 31.2 -> 43.6 mm
- added copper zone on F.Cu, net Net-(U2-ADJ)
