File: KiCad/Amplifier/Bias.kicad_sch (KiCad schematic)
At the start: 14 parts

Commit message: Platinenentwurf
die Platine wurde aufgebaut. Kontrolle fehlt
Parts:
- renumbered RV2 to RV1, RV1 to RV2
Changed lines of the file:
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@@
 		(on_board yes)
 		(dnp no)
-		(property "Reference" "RV1"
+		(property "Reference" "RV2"
 			(at 118.11 104.648 90)
 			(effects
@@
 			(project "Amplifier"
 				(path "/959c1323-2e5d-4cfd-bd7b-6fba2b4a12d5/ac42f7f1-e0b6-4538-8522-56dbee4978de"
-					(reference "RV1")
+					(reference "RV2")
 					(unit 1)
 				)
@@
 		(on_board yes)
 		(dnp no)
-		(property "Reference" "RV2"
+		(property "Reference" "RV1"
 			(at 128.27 83.058 90)
 			(effects
@@
 			(project "Amplifier"
 				(path "/959c1323-2e5d-4cfd-bd7b-6fba2b4a12d5/ac42f7f1-e0b6-4538-8522-56dbee4978de"
-					(reference "RV2")
-					(unit 1)
-				)
+					(reference "RV1")
+					(unit 1)
+				)
