File: KiCad/Amplifier/OPV2.kicad_sch (KiCad schematic)
At the start: 52 parts, among them Q10 BD140, Q7 BD139, Q8 BD139, Q9 BD140, U1 AD8017ARZ

Commit message: Platinenentwurf
die Platine wurde aufgebaut. Kontrolle fehlt
Parts:
- C126, C140, C26, C29, C37, C40: footprint Capacitor_SMD:C_0603_1608Metric_Pad1.08x0.95mm_HandSolder -> Capacitor_SMD:C_1210_3225Metric_Pad1.33x2.70mm_HandSolder
- renumbered R44 to R30, R41 to R37, R37 to R41, R30 to R44
Connections:
- net at C141.2, Q7.1 (E), R30.2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: now also Q9.1 (E); no longer Q9.2 (C)
- net at C40.1, C43.1, R53.2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: now also Q10.2 (C); no longer Q10.1 (E)
- net at C140.1, C44.1, R54.2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: now also Q9.2 (C); no longer Q9.1 (E)
- net at Q8.1 (E), R28.2, R29.2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: now also Q10.1 (E); no longer Q10.2 (C)
Changed lines of the file:
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@@
 		(on_board yes)
 		(dnp no)
-		(property "Reference" "R30"
+		(property "Reference" "R44"
 			(at 151.384 141.986 90)
 			(effects
@@
 			(project "Amplifier"
 				(path "/959c1323-2e5d-4cfd-bd7b-6fba2b4a12d5/0fd92913-fffc-43bb-bffd-f9f40efdc060"
-					(reference "R30")
+					(reference "R44")
 					(unit 1)
 				)
@@
 			)
 		)
-		(property "Footprint" "Capacitor_SMD:C_0603_1608Metric_Pad1.08x0.95mm_HandSolder"
+		(property "Footprint" "Capacitor_SMD:C_1210_3225Metric_Pad1.33x2.70mm_HandSolder"
 			(at 109.5248 160.02 0)
 			(effects
@@
 		(on_board yes)
 		(dnp no)
-		(property "Reference" "R41"
+		(property "Reference" "R37"
 			(at 151.384 161.036 90)
 			(effects
@@
 			(project "Amplifier"
 				(path "/959c1323-2e5d-4cfd-bd7b-6fba2b4a12d5/0fd92913-fffc-43bb-bffd-f9f40efdc060"
-					(reference "R41")
+					(reference "R37")
 					(unit 1)
 				)
@@
 		(on_board yes)
 		(dnp no)
-		(property "Reference" "R37"
+		(property "Reference" "R41"
 			(at 151.384 152.146 90)
 			(effects
@@
 			(project "Amplifier"
 				(path "/959c1323-2e5d-4cfd-bd7b-6fba2b4a12d5/0fd92913-fffc-43bb-bffd-f9f40efdc060"
-					(reference "R37")
+					(reference "R41")
 					(unit 1)
 				)
@@
 		(lib_id "Transistor_BJT:BD140")
 		(at 101.6 156.21 0)
+		(mirror x)
 		(unit 1)
 		(exclude_from_sim no)
@@
 		(dnp no)
 		(property "Reference" "Q9"
-			(at 105.918 152.146 0)
+			(at 105.918 160.274 0)
 			(effects
 				(font
@@
 		)
 		(property "Value" "BD140"
-			(at 105.918 154.686 0)
+			(at 105.918 157.734 0)
 			(effects
 				(font
@@
 		)
 		(property "Footprint" "Package_TO_SOT_THT:TO-126-3_Vertical"
-			(at 106.68 158.115 0)
+			(at 106.68 154.305 0)
 			(effects
 				(font
@@
 		(on_board yes)
 		(dnp no)
-		(property "Reference" "R44"
+		(property "Reference" "R30"
 			(at 151.384 169.926 90)
 			(effects
@@
 			(project "Amplifier"
 				(path "/959c1323-2e5d-4cfd-bd7b-6fba2b4a12d5/0fd92913-fffc-43bb-bffd-f9f40efdc060"
-					(reference "R44")
+					(reference "R30")
 					(unit 1)
 				)
@@
 			)
 		)
-		(property "Footprint" "Capacitor_SMD:C_0603_1608Metric_Pad1.08x0.95mm_HandSolder"
+		(property "Footprint" "Capacitor_SMD:C_1210_3225Metric_Pad1.33x2.70mm_HandSolder"
 			(at 173.6852 45.72 0)
 			(effects
@@
 			)
 		)
-		(property "Footprint" "Capacitor_SMD:C_0603_1608Metric_Pad1.08x0.95mm_HandSolder"
+		(property "Footprint" "Capacitor_SMD:C_1210_3225Metric_Pad1.33x2.70mm_HandSolder"
 			(at 89.8652 86.36 0)
 			(effects
@@
 			)
 		)
-		(property "Footprint" "Capacitor_SMD:C_0603_1608Metric_Pad1.08x0.95mm_HandSolder"
+		(property "Footprint" "Capacitor_SMD:C_1210_3225Metric_Pad1.33x2.70mm_HandSolder"
 			(at 171.7548 76.2 0)
 			(effects
@@
 		(lib_id "Transistor_BJT:BD140")
 		(at 163.83 68.58 0)
+		(mirror x)
 		(unit 1)
 		(exclude_from_sim no)
@@
 		(dnp no)
 		(property "Reference" "Q10"
-			(at 168.148 64.516 0)
+			(at 168.148 72.644 0)
 			(effects
 				(font
@@
 		)
 		(property "Value" "BD140"
-			(at 168.148 67.056 0)
+			(at 168.148 70.104 0)
 			(effects
 				(font
@@
 		)
 		(property "Footprint" "Package_TO_SOT_THT:TO-126-3_Vertical"
-			(at 168.91 70.485 0)
+			(at 168.91 66.675 0)
 			(effects
 				(font
@@
 			)
 		)
-		(property "Footprint" "Capacitor_SMD:C_0603_1608Metric_Pad1.08x0.95mm_HandSolder"
+		(property "Footprint" "Capacitor_SMD:C_1210_3225Metric_Pad1.33x2.70mm_HandSolder"
 			(at 111.4552 133.35 0)
 			(effects
@@
 			)
 		)
-		(property "Footprint" "Capacitor_SMD:C_0603_1608Metric_Pad1.08x0.95mm_HandSolder"
+		(property "Footprint" "Capacitor_SMD:C_1210_3225Metric_Pad1.33x2.70mm_HandSolder"
 			(at 106.3752 46.99 0)
 			(effects
