File: KiCad/Projects/Amplifier2/Amplifier2.kicad_pcb (KiCad board)
At the start: 4 copper layers, 255.3 x 117.9 mm, 200 parts, among them J1 Input, J2 Enable, J3 Vp_8V, J4 Vn_-5V, J5 Output, J6 Input_56V, Q1 BD139, Q10 BD140, Q2 IXTH90P10P, Q4 BD139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

Commit message: update
completed design and parts
Parts:
- removed R1.1: 10k, Resistor_SMD:R_0603_1608Metric_Pad0.98x0.95mm_HandSolder
- removed R1.2: 2k, Resistor_SMD:R_0603_1608Metric_Pad0.98x0.95mm_HandSolder
- added RP1: R_Potentiometer, Library:PVG3A, F.Cu at (119.5, 120.7)
- added RP2: R_Potentiometer, Library:PVG3A, F.Cu at (127.5, 120.7)
- CT16: value 10u -> 10n
- CT20, CT21: footprint HF:153CLV-1014 -> Capacitor_SMD:CP_Elec_10x10.5
- CT40: footprint HF:E5-13 -> Capacitor_THT:CP_Radial_D12.5mm_P5.00mm
- R2, R45, R46, R48, R49: footprint Resistor_SMD:R_0603_1608Metric_Pad0.98x0.95mm_HandSolder -> Resistor_SMD:R_1210_3225Metric_Pad1.30x2.65mm_HandSolder
- RV1: value R_Potentiometer -> 10k; footprint Library:PVG3A -> Resistor_SMD:R_0603_1608Metric_Pad0.98x0.95mm_HandSolder
- RV2: value R_Potentiometer -> 2k; footprint Library:PVG3A -> Resistor_SMD:R_0603_1608Metric_Pad0.98x0.95mm_HandSolder
- moved RV2 84.8 mm to (42.7, 124.5), turned to 0 degrees
- moved RV1 76.7 mm to (42.7, 122.9)
- moved TR3 27.6 mm to (180.1, 43.8)
- moved TR2 26.9 mm to (179.6, 121.7)
- moved K1 12.5 mm to (264.5, 78.8)
- moved T1S3 7.65 mm to (144.8, 86.1), turned to 90 degrees
- moved T1P4 7.40 mm to (144.8, 78.5), turned to -90 degrees
- moved CT35 3.92 mm to (200.6, 101.1)
- moved CT36 3.92 mm to (200.6, 97.5)
- moved CT39 3.92 mm to (200.6, 86.9)
- moved CT37 3.92 mm to (200.6, 94.0)
- moved CT38 3.92 mm to (200.6, 90.4)
- moved U3 3.63 mm to (131.5, 65.2)
- moved CT32 3.61 mm to (200.1, 71.6)
- moved CT34 3.61 mm to (200.1, 64.5)
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Connections:
- RV1 pad 1: Net-(C1-Pad1) -> /Switch/ENA
- RV1 pad 2: Net-(R14-Pad2) -> Net-(U4--)
- RV2 pad 1: Net-(C1-Pad1) -> Net-(U4--)
- RV2 pad 2: Net-(R17-Pad2) -> GND
Routing:
- net Enable: track 369.4 -> 417.0 mm
- net Net-(J4-Pin_1): track 24.2 -> 21.0 mm
- net Net-(C34-Pad2): track 6.29 -> 9.18 mm
- net Output_56V: track 214.3 -> 216.3 mm
- net Input_Signal: track 53.5 -> 51.6 mm
- net GND: track 205.1 -> 206.9 mm
- net Input_56V: track 132.0 -> 130.8 mm
- net Vn: track 109.5 -> 108.2 mm
- net Net-(D5-K-Pad3): track 8.85 -> 10.1 mm
- net Vp: track 235.0 -> 236.1 mm
- net Net-(J3-Pin_1): track 19.7 -> 20.4 mm
- net Net-(U1--VS): track 13.5 -> 14.1 mm
- net Net-(D1-K): track 19.5 -> 20.1 mm
- net Net-(Q7-C): track 22.9 -> 22.4 mm
Other:
- board text added: "HF Verstärker Ver 0.1 FH Dortmund Mohamad Sayad"
