File: KiCad/Projects/Amplifier2/HF_Part.kicad_sch (KiCad schematic)
At the start: 59 parts, among them J5 Output, T1P3 THICKPINSMD2,5X4, T1P4 THICKPINSMD2,5X4, T1S3 THICKPINSMD2,5X4, T1S4 THICKPINSMD2,5X4, U3 BLF188XRU, U6 LT1085-12

Commit message: update
completed design and parts
Parts:
- CT16: value 10u -> 10n
- CT20, CT21: footprint HF:153CLV-1014 -> Capacitor_SMD:CP_Elec_10x10.5
- CT40: footprint HF:E5-13 -> Capacitor_THT:CP_Radial_D12.5mm_P5.00mm
Other:
- moved on the sheet: C20
Changed lines of the file:
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@@
 	)
 	(junction
-		(at 74.93 167.64)
-		(diameter 0)
-		(color 0 0 0 0)
-	)
-	(junction
 		(at 21.59 99.06)
 		(diameter 0)
@@
 		(color 0 0 0 0)
 	)
+	(junction
+		(at 74.93 168.91)
+		(diameter 0)
+		(color 0 0 0 0)
+	)
 	(wire
 		(pts
@@
 	(wire
 		(pts
-			(xy 74.93 167.64) (xy 74.93 168.91)
+			(xy 74.93 153.67) (xy 74.93 168.91)
 		)
 		(stroke
@@
 	(wire
 		(pts
-			(xy 58.42 177.8) (xy 58.42 175.26)
+			(xy 58.42 177.8) (xy 58.42 176.53)
 		)
 		(stroke
@@
 	(wire
 		(pts
-			(xy 74.93 153.67) (xy 74.93 167.64)
-		)
-		(stroke
-			(width 0)
-			(type default)
-		)
-	)
-	(wire
-		(pts
 			(xy 250.19 49.53) (xy 259.08 49.53)
 		)
@@
 	(wire
 		(pts
-			(xy 58.42 167.64) (xy 74.93 167.64)
+			(xy 58.42 168.91) (xy 74.93 168.91)
 		)
 		(stroke
@@
 	)
 	(label "RFB1"
-		(at 68.58 167.64 0)
+		(at 68.58 168.91 0)
 		(fields_autoplaced yes)
 		(effects
@@
 	(symbol
 		(lib_id "Device:C")
-		(at 58.42 171.45 180)
+		(at 58.42 172.72 180)
 		(unit 1)
 		(exclude_from_sim no)
@@
 		(dnp no)
 		(property "Reference" "C20"
-			(at 55.626 170.434 0)
+			(at 55.626 171.704 0)
 			(effects
 				(font
@@
 		)
 		(property "Value" "1nF"
-			(at 55.626 172.212 0)
+			(at 55.626 173.482 0)
 			(effects
 				(font
@@
 		)
 		(property "Footprint" "Capacitor_SMD:C_0603_1608Metric_Pad1.08x0.95mm_HandSolder"
-			(at 57.4548 167.64 0)
+			(at 57.4548 168.91 0)
 			(effects
 				(font
@@
 		)
 		(property "Datasheet" "~"
-			(at 58.42 171.45 0)
+			(at 58.42 172.72 0)
 			(effects
 				(font
@@
 		)
 		(property "Description" "Unpolarized capacitor"
-			(at 58.42 171.45 0)
+			(at 58.42 172.72 0)
 			(effects
 				(font
@@
 			)
 		)
-		(property "Footprint" "HF:E5-13"
+		(property "Footprint" "Capacitor_THT:CP_Radial_D12.5mm_P5.00mm"
 			(at 68.8848 25.4 0)
 			(effects
@@
 			)
 		)
-		(property "Value" "10u"
+		(property "Value" "10n"
 			(at 53.848 100.838 0)
 			(effects
@@
 			)
 		)
-		(property "Footprint" "HF:153CLV-1014"
+		(property "Footprint" "Capacitor_SMD:CP_Elec_10x10.5"
 			(at 49.53 56.8452 0)
 			(effects
@@
 			)
 		)
-		(property "Footprint" "HF:153CLV-1014"
+		(property "Footprint" "Capacitor_SMD:CP_Elec_10x10.5"
 			(at 21.59 110.1852 0)
 			(effects
