File: KiCad/Projects/Amplifier2/OPV2.kicad_sch (KiCad schematic)
At the start: 52 parts, among them Q10 BD140, Q7 BD139, Q8 BD139, Q9 BD140, U1 AD8017ARZ

Commit message: update
completed design and parts
Changed lines of the file:
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@@
 		(dnp no)
 		(property "Reference" "Q10"
-			(at 168.148 72.644 0)
+			(at 169.672 68.072 0)
 			(effects
 				(font
