File: KiCad/Projects/Amplifier2/Switch.kicad_sch (KiCad schematic)
At the start: 43 parts, among them Q1 BD139, Q2 IXTH90P10P, Q4 BD139, Q5A1 BSC340N08NS3G, Q6 BD139, U4 AD8033, U5 LT3014xS5

Commit message: update
completed design and parts
Parts:
- R2: footprint Resistor_SMD:R_0603_1608Metric_Pad0.98x0.95mm_HandSolder -> Resistor_SMD:R_1210_3225Metric_Pad1.30x2.65mm_HandSolder
- renumbered R1.1 to RV1, R1.2 to RV2
Changed lines of the file:
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@@
 			)
 		)
-		(property "Footprint" "Resistor_SMD:R_0603_1608Metric_Pad0.98x0.95mm_HandSolder"
+		(property "Footprint" "Resistor_SMD:R_1210_3225Metric_Pad1.30x2.65mm_HandSolder"
 			(at 94.742 74.93 90)
 			(effects
@@
 		(dnp no)
 		(fields_autoplaced yes)
-		(property "Reference" "R1.2"
-			(at 78.74 118.11 0)
+		(property "Reference" "RV2"
+			(at 78.74 118.1099 0)
 			(effects
 				(font
@@
 		)
 		(property "Value" "2k"
-			(at 78.74 120.65 0)
+			(at 78.74 120.6499 0)
 			(effects
 				(font
@@
 			(project "Amplifier"
 				(path "/959c1323-2e5d-4cfd-bd7b-6fba2b4a12d5/911c4e90-f560-4b90-b362-2a5bcb196d1c"
-					(reference "R1.2")
+					(reference "RV2")
 					(unit 1)
 				)
@@
 		(dnp no)
 		(fields_autoplaced yes)
-		(property "Reference" "R1.1"
-			(at 78.74 106.68 0)
+		(property "Reference" "RV1"
+			(at 78.74 106.6799 0)
 			(effects
 				(font
@@
 		)
 		(property "Value" "10k"
-			(at 78.74 109.22 0)
+			(at 78.74 109.2199 0)
 			(effects
 				(font
@@
 			(project "Amplifier"
 				(path "/959c1323-2e5d-4cfd-bd7b-6fba2b4a12d5/911c4e90-f560-4b90-b362-2a5bcb196d1c"
-					(reference "R1.1")
-					(unit 1)
-				)
+					(reference "RV1")
+					(unit 1)
+				)
